Commit message: Serup wheels

File: projects/03_spacecraft/urdf/spacecraft.urdf (robot description, URDF)
Before this commit: robot spacecraft, 12 links, 11 joints
Joints:
- joint bus_to_mass_1: origin xyz=0.00000000 -0.00000000 -0.00000000 rpy=0.00000000 0.00000000 0.00000000 -> xyz=-0.00000000 -0.00000000 0.55000000 rpy=0.00000000 0.00000000 0.00000000
- joint bus_to_mass_2: origin xyz=-0.00000003 0.00000003 0.00000000 rpy=0.00000000 0.00000000 0.00000000 -> xyz=0.00000003 0.00000003 0.00000000 rpy=0.00000000 0.00000000 0.00000000
- joint bus_to_mass_3: origin xyz=0.00000003 -0.00000003 -0.00000000 rpy=0.00000000 0.00000000 0.00000000 -> xyz=-0.00000003 -0.00000003 -0.00000000 rpy=0.00000000 0.00000000 0.00000000
- joint bus_to_mass_4: origin xyz=0.00000000 0.00000000 0.00000000 rpy=0.00000000 0.00000000 0.00000000 -> xyz=0.00000002 0.00000000 0.00000002 rpy=0.00000000 0.00000000 0.00000000
- joint bus_to_mass_5: origin xyz=-0.00000000 -0.00000000 -0.00000000 rpy=0.00000000 0.00000000 0.00000000 -> xyz=-0.00000002 -0.00000000 -0.00000002 rpy=0.00000000 0.00000000 0.00000000
- joint bus_to_mass_6: origin xyz=0.00000000 -0.00000001 0.00000001 rpy=0.00000000 0.00000000 0.00000000 -> xyz=0.00000000 0.00000001 0.00000001 rpy=0.00000000 0.00000000 0.00000000
- joint bus_to_mass_7: origin xyz=-0.00000000 0.00000001 -0.00000001 rpy=0.00000000 0.00000000 0.00000000 -> xyz=-0.00000000 -0.00000001 -0.00000001 rpy=0.00000000 0.00000000 0.00000000
- joint bus_to_wheel_1: origin xyz=1.55563492 1.55563492 0.00000000 rpy=1.57079633 0.00000000 2.35619449 -> xyz=1.10000000 1.90525589 0.00000000 rpy=1.57079633 0.00000000 2.61799388
- joint bus_to_wheel_2: origin xyz=-1.55563492 1.55563492 0.00000000 rpy=1.57079633 0.00000000 3.92699082 -> xyz=-2.20000000 0.00000000 0.00000000 rpy=1.57079633 0.00000000 4.71238898
- joint bus_to_wheel_3: origin xyz=-1.55563492 -1.55563492 0.00000000 rpy=1.57079633 0.00000000 5.49778714 -> xyz=1.10000000 -1.90525589 0.00000000 rpy=1.57079633 0.00000000 6.80678408
- joint bus_to_wheel_4: origin xyz=1.55563492 -1.55563492 0.00000000 rpy=1.57079633 0.00000000 7.06858347 -> xyz=0.00000000 0.00000000 -2.20000000 rpy=3.14159265 0.00000000 1.57079633

Commit message: update wheels

File: projects/03_spacecraft/urdf/spacecraft.urdf (robot description, URDF)
Before this commit: robot spacecraft, 12 links, 11 joints
Joints:
- joint bus_to_mass_1: origin xyz=-0.00000000 -0.00000000 0.55000000 rpy=0.00000000 0.00000000 0.00000000 -> xyz=-0.00000000 -0.00000000 -0.27500000 rpy=0.00000000 0.00000000 0.00000000
- joint bus_to_mass_2: origin xyz=0.00000003 0.00000003 0.00000000 rpy=0.00000000 0.00000000 0.00000000 -> xyz=0.00000002 0.00000002 0.00000000 rpy=0.00000000 0.00000000 0.00000000
- joint bus_to_mass_3: origin xyz=-0.00000003 -0.00000003 -0.00000000 rpy=0.00000000 0.00000000 0.00000000 -> xyz=-0.00000002 -0.00000002 -0.00000000 rpy=0.00000000 0.00000000 0.00000000
- joint bus_to_mass_4: origin xyz=0.00000002 0.00000000 0.00000002 rpy=0.00000000 0.00000000 0.00000000 -> xyz=0.00000001 0.00000000 0.00000001 rpy=0.00000000 0.00000000 0.00000000
- joint bus_to_mass_5: origin xyz=-0.00000002 -0.00000000 -0.00000002 rpy=0.00000000 0.00000000 0.00000000 -> xyz=-0.00000001 -0.00000000 -0.00000001 rpy=0.00000000 0.00000000 0.00000000
- joint bus_to_mass_6: origin xyz=0.00000000 0.00000001 0.00000001 rpy=0.00000000 0.00000000 0.00000000 -> xyz=0.00000000 -0.00000002 0.00000002 rpy=0.00000000 0.00000000 0.00000000
- joint bus_to_mass_7: origin xyz=-0.00000000 -0.00000001 -0.00000001 rpy=0.00000000 0.00000000 0.00000000 -> xyz=-0.00000000 0.00000002 -0.00000002 rpy=0.00000000 0.00000000 0.00000000
- joint bus_to_wheel_1: origin xyz=1.10000000 1.90525589 0.00000000 rpy=1.57079633 0.00000000 2.61799388 -> xyz=0.95262794 1.65000000 1.10000000 rpy=1.04719755 0.00000000 2.61799388
- joint bus_to_wheel_2: origin xyz=-2.20000000 0.00000000 0.00000000 rpy=1.57079633 0.00000000 4.71238898 -> xyz=-1.90525589 0.00000000 1.10000000 rpy=1.04719755 0.00000000 4.71238898
- joint bus_to_wheel_3: origin xyz=1.10000000 -1.90525589 0.00000000 rpy=1.57079633 0.00000000 6.80678408 -> xyz=0.95262794 -1.65000000 1.10000000 rpy=1.04719755 0.00000000 6.80678408
